Commit message: Passing robot name to rviz models

File: vehicles/descriptions/brov2heavy_description/urdf/brov2heavy.urdf.xacro (robot description, xacro)
@@ -9,5 +9,5 @@
       <!-- <origin xyz="0. 0 0." rpy="${-pi/2} ${-pi/2} 0"/> -->
       <!-- <origin xyz="0. 0 0." rpy="0 0 0"/> -->
-      <origin xyz="0. 0. 0." rpy="0. 0. 0."/>
+      <origin xyz="0. 0. 0." rpy="${pi} 0. 0."/>
       <geometry>
         <mesh filename="${body}" scale="1 1 1"/>
