Commit message: Not being used. Reverted

File: vehicles/descriptions/sam_description/urdf/sam_auv.urdf.xacro (robot description, xacro)
@@ -6,8 +6,7 @@
   <xacro:property name="front_prop" value="file://$(find sam_description)/mesh/SAM_FRONTPROP.dae"/>
   <xacro:property name="back_prop" value="file://$(find sam_description)/mesh/SAM_BACKPROP.dae"/>
-  <xacro:property name="ns" value="sam"/>
   <xacro:macro name="sam_auv" params="debug">
   <!-- Links. -->
-  <link name="${ns}/base_link">
+  <link name="base_link">
     <visual>
       <origin xyz="-0.677 0 0" rpy="0 0 0"/>
@@ -17,5 +16,5 @@
     </visual>
   </link>
-  <link name="${ns}/thruster_link">
+  <link name="thruster_link">
     <visual>
       <origin xyz="0 0 0" rpy="0 0 0"/>
@@ -25,5 +24,5 @@
     </visual>
   </link>
-  <link name="${ns}/front_prop_link">
+  <link name="front_prop_link">
     <visual>
       <origin xyz="0 0 0" rpy="0 0 0"/>
@@ -33,5 +32,5 @@
     </visual>
   </link>
-  <link name="${ns}/back_prop_link">
+  <link name="back_prop_link">
     <visual>
       <origin xyz="0 0 0" rpy="0 0 0"/>
@@ -41,22 +40,22 @@
     </visual>
   </link>
-  <link name="${ns}/thruster_yaw_link"/>
-  <link name="${ns}/battery_link"/>
-  <link name="${ns}/tcg1_link"/>
-  <link name="${ns}/tcg2_link"/>
-  <link name="${ns}/pressure_link"/>
-  <link name="${ns}/dvl_link"/>
-  <link name="${ns}/sidescan_link"/>
-  <link name="${ns}/imu_link"/>
-  <link name="${ns}/sbg_link"/>
-  <link name="${ns}/gps_link"/>
-  <link name="${ns}/uw_gps_link"/>
-  <link name="${ns}/camera_down_link"/>
-  <link name="${ns}/camera_front_right_link"/>
-  <link name="${ns}/camera_front_left_link"/>
-  <link name="${ns}/camera_front_link"/>
+  <link name="thruster_yaw_link"/>
+  <link name="battery_link"/>
+  <link name="tcg1_link"/>
+  <link name="tcg2_link"/>
+  <link name="pressure_link"/>
+  <link name="dvl_link"/>
+  <link name="sidescan_link"/>
+  <link name="imu_link"/>
+  <link name="sbg_link"/>
+  <link name="gps_link"/>
+  <link name="uw_gps_link"/>
+  <link name="camera_down_link"/>
+  <link name="camera_front_right_link"/>
+  <link name="camera_front_left_link"/>
+  <link name="camera_front_link"/>
   <joint name="thruster_yaw_joint" type="revolute">
-    <parent link="${ns}/base_link"/>
-    <child link="${ns}/thruster_yaw_link"/>
+    <parent link="base_link"/>
+    <child link="thruster_yaw_link"/>
     <origin rpy="0.0 0.0 0.0" xyz="-0.677 0.0 0.0"/>
     <axis xyz="0 0 1"/>
@@ -64,6 +63,6 @@
   </joint>
   <joint name="thruster_pitch_joint" type="revolute">
-    <parent link="${ns}/thruster_yaw_link"/>
-    <child link="${ns}/thruster_link"/>
+    <parent link="thruster_yaw_link"/>
+    <child link="thruster_link"/>
     <origin rpy="0.0 0.0 0.0" xyz="0.0 0.0 0.0"/>
     <axis xyz="0 1 0"/>
@@ -71,76 +70,76 @@
   </joint>
   <joint name="front_prop_joint" type="continuous">
-    <parent link="${ns}/base_link"/>
-    <child link="${ns}/front_prop_link"/>
+    <parent link="base_link"/>
+    <child link="front_prop_link"/>
     <origin rpy="0.0 0.0 0.0" xyz="-0.733 0 0"/>
     <axis xyz="1 0 0"/>
   </joint>
   <joint name="back_prop_joint" type="continuous">
-    <parent link="${ns}/base_link"/>
-    <child link="${ns}/back_prop_link"/>
+    <parent link="base_link"/>
+    <child link="back_prop_link"/>
     <origin rpy="0.0 0.0 0.0" xyz="-0.751 0 0"/>
     <axis xyz="1 0 0"/>
   </joint>
   <joint name="pressure_joint" type="fixed">
-    <parent link="${ns}/base_link"/>
-    <child link="${ns}/pressure_link"/>
+    <parent link="base_link"/>
+    <child link="pressure_link"/>
     <origin rpy="0.0 0.0 0.0" xyz="-0.503 0.025 0.057"/>
   </joint>
   <joint name="dvl_joint" type="fixed">
-    <parent link="${ns}/base_link"/>
-    <child link="${ns}/dvl_link"/>
+    <parent link="base_link"/>
+    <child link="dvl_link"/>
     <origin rpy="0.0 0.0 0.0" xyz="0.573 0.0 -0.063"/>
   </joint>
   <!--Sidescan acoustic center, i.e. intersection between both sidescan centers.-->
   <joint name="sidescan_joint" type="fixed">
-    <parent link="${ns}/base_link"/>
-    <child link="${ns}/sidescan_link"/>
+    <parent link="base_link"/>
+    <child link="sidescan_link"/>
     <origin rpy="0.0 0.0 0.0" xyz="-0.043 0.0 0.0"/>
   </joint>
   <joint name="imu_joint" type="fixed">
-    <parent link="${ns}/base_link"/>
-    <child link="${ns}/imu_link"/>
+    <parent link="base_link"/>
+    <child link="imu_link"/>
     <origin rpy="0.0 0.0 0.0" xyz="0.24 0.0 -0.036"/>
   </joint>
   <joint name="sbg_joint" type="fixed">
-    <parent link="${ns}/base_link"/>
-    <child link="${ns}/sbg_link"/>
+    <parent link="base_link"/>
+    <child link="sbg_link"/>
     <origin rpy="0.0 0.0 0.0" xyz="0.46 0.0 0.002"/>
   </joint>
   <joint name="gps_joint" type="fixed">
-    <parent link="${ns}/base_link"/>
-    <child link="${ns}/gps_link"/>
+    <parent link="base_link"/>
+    <child link="gps_link"/>
     <origin rpy="0.0 0.0 0.0" xyz="0.528 0.0 0.071"/>
   </joint>
   <joint name="uw_gps_joint" type="fixed">
-    <parent link="${ns}/base_link"/>
-    <child link="${ns}/uw_gps_link"/>
+    <parent link="base_link"/>
+    <child link="uw_gps_link"/>
     <origin rpy="0.0 0.0 0.0" xyz="-0.402 0.0 0.078"/>
   </joint>
   <!-- Waterlink Nosecone Camera Positions -->
   <joint name="camera_front_joint" type="fixed">
-    <parent link="${ns}/base_link"/>
-    <child link="${ns}/camera_front_link"/>
+    <parent link="base_link"/>
+    <child link="camera_front_link"/>
     <origin rpy="-1.5707 0.0 -1.5707" xyz="0.647 0.0 0.0"/>
   </joint>
   <joint name="camera_down_joint" type="fixed">
-    <parent link="${ns}/base_link"/>
-    <child link="${ns}/camera_down_link"/>
+    <parent link="base_link"/>
+    <child link="camera_down_link"/>
     <origin rpy="3.1416 0.0 -1.5707" xyz="0.5905 0.0 -0.058"/>
   </joint>
   <joint name="camera_front_left_joint" type="fixed">
-    <parent link="${ns}/base_link"/>
-    <child link="${ns}/camera_front_left_link"/>
+    <parent link="base_link"/>
+    <child link="camera_front_left_link"/>
     <!--origin rpy="1.3 3.1416 2.3416" xyz="0.636 0.050 -0.007"/-->
     <origin rpy="1.3 3.1416 2.3416" xyz="0.636 0.050 -0.007"/>
   </joint>
   <joint name="camera_front_right_joint" type="fixed">
-    <parent link="${ns}/base_link"/>
-    <child link="${ns}/camera_front_right_link"/>
+    <parent link="base_link"/>
+    <child link="camera_front_right_link"/>
     <origin rpy="1.3 3.1416 0.8" xyz="0.636 -0.050 -0.007"/>
   </joint>
   <joint name="lcg_joint" type="prismatic">
-    <parent link="${ns}/base_link"/>
-    <child link="${ns}/battery_link"/>
+    <parent link="base_link"/>
+    <child link="battery_link"/>
     <origin rpy="0.0 0.0 0.0" xyz="0.083 0.0 0.0"/>
     <axis xyz="1 0 0"/>
@@ -148,6 +147,6 @@
   </joint>
   <joint name="tcg_joint1" type="revolute">
-    <parent link="${ns}/base_link"/>
-    <child link="${ns}/tcg1_link"/>
+    <parent link="base_link"/>
+    <child link="tcg1_link"/>
     <origin rpy="0.0 0.0 0.0" xyz="-0.095 0.0 0.0"/>
     <axis xyz="1 0 0"/>
@@ -155,6 +154,6 @@
   </joint>
   <joint name="tcg_joint2" type="revolute">
-    <parent link="${ns}/base_link"/>
-    <child link="${ns}/tcg2_link"/>
+    <parent link="base_link"/>
+    <child link="tcg2_link"/>
     <origin rpy="0.0 0.0 0.0" xyz="-0.125 0.0 0.0"/>
     <axis xyz="1 0 0"/>
