Commit message: Added geofence nodes to evolo_bringup and changed tf to z1 camera tree is connected to the rest

File: vehicles/descriptions/evolo_description/urdf/evolo.urdf (robot description, URDF)
Before this commit: robot evolo, 6 links, 5 joints
Links:
- removed link evolo/gimbal/z1_base
- added link evolo/z1_base_link
Joints:
- joint evolo/camera_joint: child evolo/gimbal/z1_base -> evolo/z1_base_link
