Commit message: lolo urdf updated + tuper controller modifications

File: vehicles/descriptions/lolo_description/urdf/lolo_auv.urdf (robot description, URDF)
Before this commit: robot lolo_auv, 18 links, 17 joints
Links:
- added link lolo/modem_link
Joints:
- added joint lolo/modem_joint: type fixed, parent lolo/base_link, child lolo/modem_link, origin xyz=1.8203 0.0016 0.7302 rpy=0 0 0
- joint lolo/usbl_joint: origin xyz=0.389 0.002 0.337 rpy=0 0 0 -> xyz=1.6103 0.0966 0.4802 rpy=0 0 0

Commit message: urdf change

File: vehicles/descriptions/lolo_description/urdf/lolo_auv.urdf (robot description, URDF)
Before this commit: robot lolo_auv, 19 links, 18 joints
Joints:
- joint lolo/modem_joint: origin xyz=1.8203 0.0016 0.7302 rpy=0 0 0 -> xyz=1.8203 0.0 0.7302 rpy=0 0 0
