Commit message: Changed lolo description to prefix frames by the parameter robot_name

File: vehicles/descriptions/lolo_description/urdf/lolo_auv.urdf (robot description, URDF)
Before this commit: robot lolo_auv, 19 links, 18 joints
Links:
- removed link lolo/base_link
- removed link lolo/compass_link
- removed link lolo/dvl_link
- removed link lolo/elevator
- removed link lolo/elevon_port
- removed link lolo/elevon_stbd
- removed link lolo/enu/mbes_link
- removed link lolo/fls_link
- removed link lolo/gps_link
- removed link lolo/imu_link
- removed link lolo/mbes_link
- removed link lolo/modem_link
- removed link lolo/pose_sensor_link
- removed link lolo/pressure_link
- removed link lolo/rudder_port
- removed link lolo/rudder_stbd
- removed link lolo/thruster_port
- removed link lolo/thruster_stbd
- removed link lolo/usbl_link
- added link base_link; visual mesh filename=file:///home/julian/colcon_ws/install/lolo_description/shar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 scale=1 1 1
- added link compass_link
- added link dvl_link
- added link elevator; visual mesh filename=file:///home/julian/colcon_ws/install/lolo_description/shar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 scale=1 1 1
- added link elevon_port; visual mesh filename=file:///home/julian/colcon_ws/install/lolo_description/shar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 scale=1 1 1
- added link elevon_stbd; visual mesh filename=file:///home/julian/colcon_ws/install/lolo_description/shar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 scale=1 1 1
- added link enu/mbes_link
- added link fls_link
- added link gps_link
- added link imu_link
- added link mbes_link
- added link modem_link
- added link pose_sensor_link; visual box size=0.01 0.01 0.01
- added link pressure_link
- added link rudder_port; visual mesh filename=file:///home/julian/colcon_ws/install/lolo_description/shar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 scale=1 1 1
- added link rudder_stbd; visual mesh filename=file:///home/julian/colcon_ws/install/lolo_description/shar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 scale=1 1 1
- added link thruster_port; visual mesh filename=file:///home/julian/colcon_ws/install/lolo_description/shar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 scale=1 1 1
- added link thruster_stbd; visual mesh filename=file:///home/julian/colcon_ws/install/lolo_description/shar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 scale=1 1 1
- added link usbl_link
Joints:
- removed joint lolo/compass_joint
- removed joint lolo/dvl_joint
- removed joint lolo/elevator_joint
- removed joint lolo/elevon_port_joint
- removed joint lolo/elevon_stbd_joint
- removed joint lolo/enu/mbes_joint
- removed joint lolo/fls_joint
- removed joint lolo/gps_joint
- removed joint lolo/imu_joint
- removed joint lolo/mbes_joint
- removed joint lolo/modem_joint
- removed joint lolo/pose_sensor_joint
- removed joint lolo/pressure_joint
- removed joint lolo/rudder_port_joint
- removed joint lolo/rudder_stbd_joint
- removed joint lolo/thruster_port_joint
- removed joint lolo/thruster_stbd_joint
- removed joint lolo/usbl_joint
- added joint compass_joint: type fixed, parent base_link, child compass_link, origin xyz=0 0 0 rpy=0 0 0
- added joint dvl_joint: type fixed, parent base_link, child dvl_link, origin xyz=0.805 -0.025 -0.245 rpy=3.14159 0 0
- added joint elevator_joint: type revolute, parent base_link, child elevator, origin xyz=-0.6476 0.0 0.0135 rpy=0 0 0, axis 0 1 0, limit lower=-0.7853981633974483 upper=0.7853981633974483 effort=0 velocity=0
- added joint elevon_port_joint: type revolute, parent base_link, child elevon_port, origin xyz=-0.3733 0.4035 0.01349 rpy=0 0 0.19652, axis 0 1 0, limit lower=-0.7853981633974483 upper=0.7853981633974483 effort=0 velocity=0
- added joint elevon_stbd_joint: type revolute, parent base_link, child elevon_stbd, origin xyz=-0.3733 -0.4035 0.01349 rpy=0 0 -0.19652, axis 0 1 0, limit lower=-0.7853981633974483 upper=0.7853981633974483 effort=0 velocity=0
- added joint enu/mbes_joint: type fixed, parent base_link, child enu/mbes_link, origin xyz=2.523 0.0155 -0.302 rpy=0 0 0
- added joint fls_joint: type fixed, parent base_link, child fls_link, origin xyz=0 0 0 rpy=0 0 0
- added joint gps_joint: type fixed, parent base_link, child gps_link, origin xyz=0.836 0 0.44 rpy=0 0 0
- added joint imu_joint: type fixed, parent base_link, child imu_link, origin xyz=0 0 0 rpy=3.14159 0 0
- added joint mbes_joint: type fixed, parent base_link, child mbes_link, origin xyz=-.751 -0.0155 0.084 rpy=0 0 0
- added joint modem_joint: type fixed, parent base_link, child modem_link, origin xyz=1.8203 0.0 0.7302 rpy=0 0 0
- added joint pose_sensor_joint: type revolute, parent base_link, child pose_sensor_link, origin xyz=0 0 0 rpy=0 0 0, limit lower=0 upper=0 effort=0 velocity=0
- added joint pressure_joint: type fixed, parent base_link, child pressure_link, origin xyz=0 0 0 rpy=0 0 0
- added joint rudder_port_joint: type revolute, parent base_link, child rudder_port, origin xyz=-0.3278 0.253 0.129 rpy=0 0 0, axis 0 0 1, limit lower=-0.7853981633974483 upper=0.7853981633974483 effort=0 velocity=0
- added joint rudder_stbd_joint: type revolute, parent base_link, child rudder_stbd, origin xyz=-0.3278 -0.253 0.129 rpy=0 0 0, axis 0 0 1, limit lower=-0.7853981633974483 upper=0.7853981633974483 effort=0 velocity=0
- added joint thruster_port_joint: type continuous, parent base_link, child thruster_port, origin xyz=-0.9056 0.2754 0.013678 rpy=0 0 0, axis 1 0 0
- added joint thruster_stbd_joint: type continuous, parent base_link, child thruster_stbd, origin xyz=-0.9056 -0.2754 0.013678 rpy=0 0 0, axis 1 0 0
- added joint usbl_joint: type fixed, parent base_link, child usbl_link, origin xyz=1.6103 0.0966 0.4802 rpy=0 0 0

Commit message: update fls_link, added oculus_link, remove deprecated enu/mbes_link

File: vehicles/descriptions/lolo_description/urdf/lolo_auv.urdf (robot description, URDF)
Before this commit: robot lolo_auv, 19 links, 18 joints
Links:
- removed link enu/mbes_link
- added link oculus_link
Joints:
- removed joint enu/mbes_joint
- added joint oculus_joint: type fixed, parent base_link, child oculus_link, origin xyz=2.2928 0.0118 0.0102 rpy=0 0.2618 0
- joint fls_joint: origin xyz=0 0 0 rpy=0 0 0 -> xyz=2.263 -0.003 0.17 rpy=1.5708 0.2443 0
